Commit message: adding action charger in pddl and action node

File: robot_urdf/urdf/robot5.xacro (robot description, xacro)
@@ -40,5 +40,5 @@
     <color rgba="1.0 1.0 1.0 1.0"/>
   </material>
-	  <link name="link_chassis">
+	<link name="link_chassis">
     <!-- pose and inertial -->
     <pose>0 0 0.1 0 0 0</pose>
@@ -75,5 +75,5 @@
     </visual>
   </link>
-   <link name="link_right_wheel">
+  <link name="link_right_wheel">
     <xacro:default_inertial mass="0.2"/>
     <collision name="link_right_wheel_collision">
@@ -87,5 +87,5 @@
     </visual>
   </link>
-   <link name="link_left_wheel">
+  <link name="link_left_wheel">
     <xacro:default_inertial mass="0.2"/>
     <collision name="link_left_wheel_collision">
@@ -116,30 +116,51 @@
   </joint>
   <link name="camera_link">
-	    <collision>
-	      <origin xyz="0 0 0.1" rpy="0 0 0"/>
-	      <geometry>
-		<box size="0.05 0.05 0.2"/>
-	      </geometry>
-	    </collision>
-	    <visual>
-	      <origin xyz="0 0 0.025" rpy="0 0 0"/>
-	      <geometry>
-		<box size="0.05 0.05 0.05"/>
-	      </geometry>
-	      <material name="red">
-		<color rgba="1 0 0 1"/>
-	      </material>
-	    </visual>
-	    <inertial>
-	      <mass value="1e-5" />
-	      <origin xyz="0 0 0" rpy="0 0 0"/>
-	      <inertia ixx="1e-6" ixy="0" ixz="0" iyy="1e-6" iyz="0" izz="1e-6" />
-	    </inertial>
+	  <collision>
+      <origin xyz="0 0 0.1" rpy="0 0 0"/>
+      <geometry>
+        <box size="0.05 0.05 0.2"/>
+      </geometry>
+	  </collision>
+	  <visual>
+	    <origin xyz="0 0 0.025" rpy="0 0 0"/>
+	    <geometry>
+		    <box size="0.05 0.05 0.05"/>
+	    </geometry>
+	    <material name="red">
+		    <color rgba="1 0 0 1"/>
+	    </material>
+	  </visual>
+	  <inertial>
+      <mass value="1e-5" />
+      <origin xyz="0 0 0" rpy="0 0 0"/>
+      <inertia ixx="1e-6" ixy="0" ixz="0" iyy="1e-6" iyz="0" izz="1e-6" />
+	  </inertial>
   </link>
   <joint name="camera_joint" type="fixed">
-	    <axis xyz="0 1 0" />
-	    <origin xyz="0.23 0 0.235" rpy="0 0 0"/>
-	    <parent link="link_chassis"/>
-	    <child link="camera_link"/>
-	 </joint>
+    <axis xyz="0 1 0" />
+    <origin xyz="0.23 0 0.235" rpy="0 0 0"/>
+    <parent link="link_chassis"/>
+    <child link="camera_link"/>
+  </joint>
+<!-- Prove per creare un nuovo link-->
+  <link name='test_link'>
+    <visual>
+      <origin xyz="0 0 0" rpy="0 0 0"/>   <!-- frame centrato con il box -->
+      <geometry>
+        <box size="0.1 0.1 0.1"/>
+      </geometry>
+      <material name="green"/>
+    </visual>
+    <collision name="collision_test_link">
+      <origin xyz="0 0 0" rpy="0 0 0"/>
+      <geometry>
+        <box size="0.1 0.1 0.1"/>
+      </geometry>
+    </collision>
+  </link>
+  <joint name="test_joint" type="fixed">
+    <parent link="link_chassis"/>
+    <child link="test_link"/>
+    <origin xyz="0.3 0 0" rpy="0 0 0"/>
+  </joint>
 </robot>
